Commit message: Renamed obj and urdf files for consistency with path npy files, updated PointMassAviary.py and pointmass.py accordingly

File: PDM_project/quadrotor_project/assets/track1.urdf (robot description, URDF)
Before this commit: robot Hole_obstacle_course.urdf, 1 links, 0 joints
Links:
- link baseLink: geometry collision mesh filename=track1.obj scale=1 1 1; visual mesh filename=track1.obj scale=1 1 1

File: PDM_project/quadrotor_project/assets/track2.urdf (robot description, URDF)
Before this commit: robot Parcour2.urdf, 1 links, 0 joints
Links:
- link baseLink: geometry collision mesh filename=track2.obj scale=1 1 1; visual mesh filename=track2.obj scale=1 1 1

File: PDM_project/quadrotor_project/assets/track3.urdf (robot description, URDF)
Before this commit: robot drone_parcours.urdf, 1 links, 0 joints
Links:
- link baseLink: geometry collision mesh filename=track3.obj scale=1 1 1; visual mesh filename=track3.obj scale=1 1 1
